Commit message: feat: Implemented deer related models and discarded leopard models.

File: packages/animal_description/urdf/animal_robot.urdf (robot description, URDF)
Before this commit: robot animal_robot, 7 links, 6 joints
Links:
- link chassis: mass 1.0 -> 3.0; geometry collision box size=0.22 0.12 0.06; visual box size=0.22 0.12 0.06
- link front_pitch_link: mass 0.001 -> 0.2; geometry collision sphere radius=0.015; visual sphere radius=0.015
- link left_wheel: mass 0.2 -> 0.3; geometry collision cylinder length=0.02 radius=0.035; visual cylinder length=0.02 radius=0.035
- link rgb_cam_camera_link: mass None -> 0.05; geometry visual box size=0.03 0.03 0.03
- link right_wheel: mass 0.2 -> 0.3; geometry collision cylinder length=0.02 radius=0.035; visual cylinder length=0.02 radius=0.035
Joints:
- joint front_pitch_joint: origin xyz=0.08 0 -0.05 rpy=0 0 0 -> xyz=0.08 0 -0.045 rpy=0 0 0
- joint joint_left_wheel: limit effort=10000 velocity=1000 -> effort=20.0 velocity=20.0; origin xyz=-0.05 -0.05 -0.025 rpy=0 0 0 -> xyz=-0.05 -0.06 -0.025 rpy=0 0 0
- joint joint_right_wheel: limit effort=10000 velocity=1000 -> effort=20.0 velocity=20.0; origin xyz=-0.05 0.05 -0.025 rpy=0 0 0 -> xyz=-0.05 0.06 -0.025 rpy=0 0 0
- joint rgb_cam_camera_link_joint: origin xyz=0.04 0.0 0.2 rpy=0 0 0 -> xyz=0.09 0.0 0.08 rpy=0 0 0
